File: 65HE_PCB/Sensors.kicad_sch (KiCad schematic)
At the start: 170 parts

Commit message: plotted schematic
exported the schematic as a PDF in order to view it in any device
Parts:
- gave numbers to parts that had none: 150
